File: PCB/SEI Photometer/SEI Photometer.kicad_pcb (KiCad board)
At the start: 2 copper layers, 33.9 x 33.9 mm, 13 parts, among them U1 MAX1674

Commit message: changed the positive and negative terminals
Routing:
- net Vin: vias 7 -> 0
- net GND: vias 0 -> 24
- added copper zone on B.Cu, net GND
- removed copper zone on B.Cu, net Vin
Changed lines of the file:
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@@
     (fp_line (start 1.525 1.525) (end -1.525 1.525)
       (stroke (width 0.12) (type solid)) (layer "F.Fab"))
-    (pad "1" smd roundrect (at -0.975 2.1 180) (size 1.171 0.4) (layers "F.Cu" "F.Paste" "F.Mask") (roundrect_rratio 0.2516986755)
+    (pad "1" smd roundrect (at -0.975 2.1 180) (size 1.171 0.4) (layers "F.Cu" "F.Paste" "F.Mask") (roundrect_rratio 0.2516975)
       (net 7 "FB") (pinfunction "FB") (pintype "input"))
-    (pad "2" smd roundrect (at -0.325 2.1 180) (size 1.171 0.4) (layers "F.Cu" "F.Paste" "F.Mask") (roundrect_rratio 0.2516986755)
+    (pad "2" smd roundrect (at -0.325 2.1 180) (size 1.171 0.4) (layers "F.Cu" "F.Paste" "F.Mask") (roundrect_rratio 0.2516975)
       (net 1 "GND") (pinfunction "LBI") (pintype "input"))
-    (pad "3" smd roundrect (at 0.325 2.1 180) (size 1.171 0.4) (layers "F.Cu" "F.Paste" "F.Mask") (roundrect_rratio 0.2516986755)
+    (pad "3" smd roundrect (at 0.325 2.1 180) (size 1.171 0.4) (layers "F.Cu" "F.Paste" "F.Mask") (roundrect_rratio 0.2516975)
       (net 9 "unconnected-(U1-~{LBO}-Pad3)") (pinfunction "~{LBO}") (pintype "input"))
-    (pad "4" smd roundrect (at 0.975 2.1 180) (size 1.171 0.4) (layers "F.Cu" "F.Paste" "F.Mask") (roundrect_rratio 0.2516986755)
+    (pad "4" smd roundrect (at 0.975 2.1 180) (size 1.171 0.4) (layers "F.Cu" "F.Paste" "F.Mask") (roundrect_rratio 0.2516975)
       (net 4 "Net-(U1-REF)") (pinfunction "REF") (pintype "input"))
-    (pad "5" smd roundrect (at 0.975 -2.1 180) (size 1.171 0.4) (layers "F.Cu" "F.Paste" "F.Mask") (roundrect_rratio 0.2516986755)
+    (pad "5" smd roundrect (at 0.975 -2.1 180) (size 1.171 0.4) (layers "F.Cu" "F.Paste" "F.Mask") (roundrect_rratio 0.2516975)
       (net 5 "Net-(D1-K)") (pinfunction "~{SHDN}") (pintype "input"))
-    (pad "6" smd roundrect (at 0.325 -2.1 180) (size 1.171 0.4) (layers "F.Cu" "F.Paste" "F.Mask") (roundrect_rratio 0.2516986755)
+    (pad "6" smd roundrect (at 0.325 -2.1 180) (size 1.171 0.4) (layers "F.Cu" "F.Paste" "F.Mask") (roundrect_rratio 0.2516975)
       (net 1 "GND") (pinfunction "GND") (pintype "input"))
-    (pad "7" smd roundrect (at -0.325 -2.1 180) (size 1.171 0.4) (layers "F.Cu" "F.Paste" "F.Mask") (roundrect_rratio 0.2516986755)
+    (pad "7" smd roundrect (at -0.325 -2.1 180) (size 1.171 0.4) (layers "F.Cu" "F.Paste" "F.Mask") (roundrect_rratio 0.2516975)
       (net 6 "Net-(D1-A)") (pinfunction "LX") (pintype "input"))
-    (pad "8" smd roundrect (at -0.975 -2.1 180) (size 1.171 0.4) (layers "F.Cu" "F.Paste" "F.Mask") (roundrect_rratio 0.2516986755)
+    (pad "8" smd roundrect (at -0.975 -2.1 180) (size 1.171 0.4) (layers "F.Cu" "F.Paste" "F.Mask") (roundrect_rratio 0.2516975)
       (net 5 "Net-(D1-K)") (pinfunction "OUT") (pintype "input"))
   )
@@
   (gr_circle (center 100 100) (end 116.95 100)
     (stroke (width 0.1) (type solid)) (fill none) (layer "Edge.Cuts"))
+  (via (at 97.75 93.85) (size 0.8) (drill 0.4) (layers "F.Cu" "B.Cu") (free) (net 1))
+  (via (at 104 106.45) (size 0.8) (drill 0.4) (layers "F.Cu" "B.Cu") (free) (net 1))
+  (via (at 98.825 93.85) (size 0.8) (drill 0.4) (layers "F.Cu" "B.Cu") (free) (net 1))
+  (via (at 95.575 106.5) (size 0.8) (drill 0.4) (layers "F.Cu" "B.Cu") (free) (net 1))
+  (via (at 101.05 106.475) (size 0.8) (drill 0.4) (layers "F.Cu" "B.Cu") (free) (net 1))
+  (via (at 106.525 96.55) (size 0.8) (drill 0.4) (layers "F.Cu" "B.Cu") (free) (net 1))
+  (via (at 92.425 106.475) (size 0.8) (drill 0.4) (layers "F.Cu" "B.Cu") (free) (net 1))
+  (via (at 102.075 106.475) (size 0.8) (drill 0.4) (layers "F.Cu" "B.Cu") (free) (net 1))
+  (via (at 106.5 95.575) (size 0.8) (drill 0.4) (layers "F.Cu" "B.Cu") (free) (net 1))
+  (via (at 105.95 93.9) (size 0.8) (drill 0.4) (layers "F.Cu" "B.Cu") (free) (net 1))
+  (via (at 100.9 93.875) (size 0.8) (drill 0.4) (layers "F.Cu" "B.Cu") (free) (net 1))
+  (via (at 94.5 106.525) (size 0.8) (drill 0.4) (layers "F.Cu" "B.Cu") (free) (net 1))
+  (via (at 98.925 106.5) (size 0.8) (drill 0.4) (layers "F.Cu" "B.Cu") (free) (net 1))
+  (via (at 97.8 106.525) (size 0.8) (drill 0.4) (layers "F.Cu" "B.Cu") (free) (net 1))
+  (via (at 103.975 93.9) (size 0.8) (drill 0.4) (layers "F.Cu" "B.Cu") (free) (net 1))
+  (via (at 99.875 93.875) (size 0.8) (drill 0.4) (layers "F.Cu" "B.Cu") (free) (net 1))
+  (via (at 103.05 106.475) (size 0.8) (drill 0.4) (layers "F.Cu" "B.Cu") (free) (net 1))
+  (via (at 96.6 106.5) (size 0.8) (drill 0.4) (layers "F.Cu" "B.Cu") (free) (net 1))
+  (via (at 96.725 93.85) (size 0.8) (drill 0.4) (layers "F.Cu" "B.Cu") (free) (net 1))
+  (via (at 104.925 93.875) (size 0.8) (drill 0.4) (layers "F.Cu" "B.Cu") (free) (net 1))
+  (via (at 102.975 93.875) (size 0.8) (drill 0.4) (layers "F.Cu" "B.Cu") (free) (net 1))
+  (via (at 93.425 106.5) (size 0.8) (drill 0.4) (layers "F.Cu" "B.Cu") (free) (net 1))
+  (via (at 101.95 93.875) (size 0.8) (drill 0.4) (layers "F.Cu" "B.Cu") (free) (net 1))
+  (via (at 100.025 106.5) (size 0.8) (drill 0.4) (layers "F.Cu" "B.Cu") (free) (net 1))
   (segment (start 90.95 92.32) (end 95.355 92.32) (width 0.9) (layer "F.Cu") (net 2))
   (segment (start 95.355 92.32) (end 95.4 92.275) (width 0.25) (layer "F.Cu") (net 2))
-  (via (at 89.6 91.1) (size 0.8) (drill 0.4) (layers "F.Cu" "B.Cu") (free) (net 2))
-  (via (at 90.5 91.1) (size 0.8) (drill 0.4) (layers "F.Cu" "B.Cu") (free) (net 2))
-  (via (at 92.35 91.1) (size 0.8) (drill 0.4) (layers "F.Cu" "B.Cu") (free) (net 2))
-  (via (at 94.15 91.1) (size 0.8) (drill 0.4) (layers "F.Cu" "B.Cu") (free) (net 2))
-  (via (at 91.4 91.1) (size 0.8) (drill 0.4) (layers "F.Cu" "B.Cu") (free) (net 2))
-  (via (at 95.05 91.1) (size 0.8) (drill 0.4) (layers "F.Cu" "B.Cu") (free) (net 2))
-  (via (at 93.25 91.1) (size 0.8) (drill 0.4) (layers "F.Cu" "B.Cu") (free) (net 2))
   (segment (start 110.025 104.925) (end 108.9 106.05) (width 0.25) (layer "F.Cu") (net 3))
   (segment (start 110.025 104.05) (end 110.025 104.925) (width 0.25) (layer "F.Cu") (net 3))
@@
   (segment (start 108.375 104.05) (end 108.375 100.025) (width 0.25) (layer "F.Cu") (net 8))
   (segment (start 108.375 100.025) (end 108.4 100) (width 0.25) (layer "F.Cu") (net 8))
-  (zone (net 2) (net_name "Vin") (layer "F.Cu") (hatch edge 0.5)
-    (priority 2)
-    (connect_pads yes (clearance 0))
-    (min_thickness 0.25) (filled_areas_thickness no)
-    (fill yes (thermal_gap 0.5) (thermal_bridge_width 0.5))
-    (polygon
-      (pts
-        (xy 89.15 93.05)
-        (xy 89.15 90.65)
-        (xy 95.9 90.65)
-        (xy 95.9 93.05)
-      )
-    )
-  )
-  (zone (net 1) (net_name "GND") (layer "F.Cu") (hatch edge 0.508)
+  (zone (net 2) (net_name "Vin") (layer "F.Cu") (hatch edge 0.508)
     (connect_pads yes (clearance 0))
     (min_thickness 0.254) (filled_areas_thickness no)
@@
   )
   (zone (net 6) (net_name "Net-(D1-A)") (layer "F.Cu") (hatch edge 0.5)
-    (priority 1)
+    (priority 2)
     (connect_pads yes (clearance 0))
     (min_thickness 0.25) (filled_areas_thickness no)
@@
     )
   )
-  (zone (net 2) (net_name "Vin") (layer "B.Cu") (name "Vin") (hatch edge 0.508)
+  (zone (net 1) (net_name "GND") (layer "F.Cu") (name "Vin") (hatch edge 0.508)
+    (priority 1)
+    (connect_pads yes (clearance 0))
+    (min_thickness 0.254) (filled_areas_thickness no)
+    (fill yes (thermal_gap 0.508) (thermal_bridge_width 0.508))
+    (polygon
+      (pts
+        (xy 93.175 93.3)
+        (xy 107.05 93.3)
+        (xy 107 106.975)
+        (xy 90.325 106.95)
+        (xy 90.325 96.925)
+        (xy 93.175 96.925)
+        (xy 93.175 93.3)
+      )
+    )
+  )
+  (zone (net 1) (net_name "GND") (layer "B.Cu") (name "Vin") (hatch edge 0.508)
     (connect_pads yes (clearance 1))
     (min_thickness 0.254) (filled_areas_thickness no)
